File: relayer.kicad_sch (KiCad schematic)
At the start: 5 parts, among them K1 SLC-12VDC-SL-C, U14 HN2199

Commit message: begin new bom
Parts:
- removed K1: SLC-12VDC-SL-C, slc-12v:RELAY-TH_SLC-XXVDC-SL-C, symbol slc-12v:SLC-12VDC-SL-C
- renumbered D2 to D3, R21 to R25, R24 to R26, U14 to U16
Connections:
- net VOUT: now also D3.1 (C)

Commit message: almost ready for prod
Parts:
- removed D3: M7F_C466485, m7f:SMAF_L3.5-W2.6-LS4.7-RD, symbol m7f:M7F_C466485
- removed R25, R26: 10K, Resistor_SMD:R_0603_1608Metric, symbol Device:R
- removed U16: HN2199, hn2199:DFN-8_L5.8-W4.9-P1.27-LS6.0-BL, symbol hn2199:HN2199
- added D1: M7F_C466485, m7f:SMAF_L3.5-W2.6-LS4.7-RD, symbol m7f:M7F_C466485
- added Q1: WSP4606, blastLib:SOP-8_L4.9-W3.9-P1.27-LS6.0-BL, symbol blastLib:WSP4606
- added R15, R16: 10K, Resistor_SMD:R_0603_1608Metric, symbol Device:R
Connections:
- net +12V: now also Q1.3 (S2), R16.1
- net DIN: now also Q1.2 (G1), R15.1
- net GND: now also Q1.1 (S1), R15.2
- net VOUT: now also D1.1 (C)
- new net: D1.2 (A), Q1.5 (D2), Q1.6 (D2)
- new net: Q1.4 (G2), Q1.7 (D1), Q1.8 (D1), R16.2

Commit message: add servo drive?
Parts:
- renumbered D1 to D3, Q1 to Q4, R15 to R23, R16 to R24
Changed lines of the file:
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@@
 		(dnp no)
 		(fields_autoplaced yes)
-		(property "Reference" "D1"
+		(property "Reference" "D3"
 			(at 182.88 63.5 0)
 			(effects
@@
 		(dnp no)
 		(fields_autoplaced yes)
-		(property "Reference" "#PWR062"
+		(property "Reference" "#PWR069"
 			(at 165.1 62.23 0)
 			(effects
@@
 		(dnp no)
 		(fields_autoplaced yes)
-		(property "Reference" "R16"
+		(property "Reference" "R24"
 			(at 160.02 66.0401 0)
 			(effects
@@
 		(dnp no)
 		(fields_autoplaced yes)
-		(property "Reference" "Q1"
+		(property "Reference" "Q4"
 			(at 171.45 45.72 90)
 			(effects
@@
 		(dnp no)
 		(fields_autoplaced yes)
-		(property "Reference" "#PWR065"
+		(property "Reference" "#PWR071"
 			(at 146.05 72.39 0)
 			(effects
@@
 		(dnp no)
 		(fields_autoplaced yes)
-		(property "Reference" "#PWR063"
+		(property "Reference" "#PWR070"
 			(at 152.4 67.31 0)
 			(effects
@@
 		(dnp no)
 		(fields_autoplaced yes)
-		(property "Reference" "R15"
+		(property "Reference" "R23"
 			(at 154.94 54.6099 0)
 			(effects
