File: relayer.kicad_sch (KiCad schematic)
At the start: 4 parts, among them Q4 WSP4606

Commit message: docs
Other:
- company: (none) -> Jet & Aeronautics Society
Changed lines of the file:
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@@
 	(title_block
 		(date "2024-04-21")
+		(company "Jet & Aeronautics Society")
 	)
 	(junction
