File: JAS Warhead PCB.kicad_sch (KiCad schematic)
At the start: 26 parts, among them J1 Conn_01x02_Socket, J2 Conn_01x02_Pin, J3 Conn_01x02_Pin, J4 Conn_01x02_Pin, J5 Conn_01x03_Pin, J6 Conn_01x03_Pin, J7 Conn_01x02_Socket, J8 Conn_01x02_Socket, U1 LD1117S50TR_SOT223, U2 DG636-7.62-02P-14-00A(H), U3 DG636-7.62-02P-14-00A(H), U4 DG636-7.62-02P-14-00A(H)

Commit message: begin new bom
Parts:
- added C27, C28: 1uF, Capacitor_SMD:C_0402_1005Metric, symbol Device:C
- added U17: AP2127R-3.3, Package_TO_SOT_SMD:SOT-89-3, symbol Regulator_Linear:AP2127R-3.3
Connections:
- net +5V: now also C27.1, U17.2 (VI)
- net 3V3: no longer J4.1 (Pin_1), R1.2, R2.1
- net GND: now also C27.2, C28.2, U17.1 (GND)
- new net +3V3: C28.1, J4.1 (Pin_1), R1.2, R2.1, U17.3 (VO)
Other:
- note added: "RELAYS ARE NOW EXTERNAL AND NOT POPULATED ON THE BOARD"
- moved on the sheet: J2, J3, J4

Commit message: almost there
Parts:
- removed J1, J7, J8: Conn_01x02_Socket, TerminalBlock:TerminalBlock_bornier-2_P5.08mm, symbol Connector:Conn_01x02_Socket
- removed J2, J4: Conn_01x02_Pin, Connector_PinHeader_2.54mm:PinHeader_1x02_P2.54mm_Vertical, symbol Connector:Conn_01x02_Pin
- removed U2, U3, U4: DG636-7.62-02P-14-00A(H), dg636:CONN-TH_DG636-7.62-02P-14-0, symbol dg636:DG636-7.62-02P-14-00A(H)
- added CN1, CN11, CN12, CN2, CN3, CN4, CN5, CN6: DB910-7.62-2P, blastLib:CONN-TH_2P-P7.62_DB910-7.62-2P, symbol blastLib:DB910-7.62-2P
- added U2: AHT20-F, blastLib:SENSOR-SMD-6_AHT20, symbol blastLib:AHT20-F
- J5, J6: now not fitted; now left out of the parts list
Connections:
- net +12V: now also CN5.2
- net +3V3: now also CN4.2, U2.2 (VDD)
- net +5V: now also CN6.2
- net GND: now also CN1.2, CN11.1, CN12.1, CN2.2, CN3.2, CN4.1, CN5.1, CN6.1, U2.5 (GND)
- net OilTemp: now also CN11.2
- net RELAY+CONTROLLER/VOUT: now also CN3.1
- net RELAY+CONTROLLER1/VOUT: now also CN2.1
- net RELAY+CONTROLLER2/VOUT: now also CN1.1
- net SCL: now also U2.3 (SCL)
- net SDA: now also U2.4 (SDA)
- net WtrTemp: now also CN12.2
- no-connect marks 0 -> 3
Other:
- sheet Load Cell ports: added SCL, SDA; removed none

Commit message: almost ready for prod
Parts:
- removed C1, C2: 10uF, Capacitor_SMD:C_0402_1005Metric, symbol Device:C
- removed C27, C28: 1uF, Capacitor_SMD:C_0402_1005Metric, symbol Device:C
- removed U1: LD1117S50TR_SOT223, Package_TO_SOT_SMD:SOT-223-3_TabPin2, symbol Regulator_Linear:LD1117S50TR_SOT223
- removed U17: AP2127R-3.3, Package_TO_SOT_SMD:SOT-89-3, symbol Regulator_Linear:AP2127R-3.3
- added C10, C3, C8: 10uF, Capacitor_SMD:C_0603_1608Metric, symbol Device:C
- added C9: 1uF, Capacitor_SMD:C_0402_1005Metric, symbol Device:C
- added U1: SE5218ALG-LF, blastLib:SOT-23-5_L3.0-W1.7-P0.95-LS2.8-BR, symbol blastLib:SE5218ALG-LF
- added U3: LM1117S-5.0, blastLib:SOT-223-3_L6.5-W3.4-P2.30-LS7.0-BR, symbol blastLib:LM1117S-5.0
Connections:
- net +12V: now also C3.1, U3.3 (IN)
- net +3V3: now also C10.1, U1.5 (VOUT)
- net +5V: now also C8.1, C9.1, U1.1 (VIN), U1.3 (ENABLE), U3.2 (OUT), U3.4 (TAB)
- net GND: now also C10.2, C3.2, C8.2, C9.2, U1.2 (GND), U3.1 (ADJ/GND)
- no-connect marks 3 -> 4

Commit message: add servo drive?
Parts:
- added J1: Conn_01x03_Pin, Connector_PinHeader_2.54mm:PinHeader_1x03_P2.54mm_Vertical, symbol Connector:Conn_01x03_Pin
Connections:
- net +5V: now also J1.1 (Pin_1)
- net GND: now also J1.3 (Pin_3)
- new net SERVO: J1.2 (Pin_2)
Other:
- note added: "TODO Remove nonsensical Diodes on SPI Lanes Re-vamp the connections for relays Connect load cell properly Re-work board placement entirely Generate BOM to work with JLC manufacturing Re-think the LDO and potentially add more power to the board Completely re-consider the size of certain things on the board, most capacitors and resistors can be 0603, except load bearing / buring resistors Add 5v Se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"
- note removed: "TODO Remove nonsensical Diodes on SPI Lanes Re-vamp the connections for relays Connect load cell properly Re-work board placement entirely Generate BOM to work with JLC manufacturing Re-think the LDO and potentially add more power to the board Completely re-consider the size of certain things on the board, most capacitors and resistors can be 0603, except load bearing / buring resistors"

Commit message: send off for prod
Changed lines of the file:
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@@
-	(wire
-		(pts
-			(xy 17.78 34.29) (xy 27.94 34.29)
-		)
-		(stroke
-			(width 0)
-			(type default)
-		)
-	)
 	(wire
 		(pts
@@
 	(wire
 		(pts
-			(xy 17.78 25.4) (xy 27.94 25.4)
-		)
-		(stroke
-			(width 0)
-			(type default)
-		)
-	)
-	(wire
-		(pts
 			(xy 109.22 172.72) (xy 115.57 172.72)
 		)
@@
 	(wire
 		(pts
+			(xy 17.78 27.94) (xy 27.94 27.94)
+		)
+		(stroke
+			(width 0)
+			(type default)
+		)
+	)
+	(wire
+		(pts
 			(xy 228.6 54.61) (xy 233.68 54.61)
 		)
@@
 		(pts
 			(xy 48.26 81.28) (xy 39.37 81.28)
+		)
+		(stroke
+			(width 0)
+			(type default)
+		)
+	)
+	(wire
+		(pts
+			(xy 17.78 38.1) (xy 27.94 38.1)
 		)
 		(stroke
@@
 		)
 	)
+	(label "SERVO"
+		(at 17.78 27.94 0)
+		(fields_autoplaced yes)
+		(effects
+			(font
+				(size 1.27 1.27)
+			)
+			(justify left bottom)
+		)
+	)
 	(label "SPI CLK"
 		(at 80.01 66.04 0)
@@
 		)
 	)
+	(label "OilTemp"
+		(at 17.78 38.1 0)
+		(fields_autoplaced yes)
+		(effects
+			(font
+				(size 1.27 1.27)
+			)
+			(justify left bottom)
+		)
+	)
 	(label "SPI CLK"
 		(at 80.01 45.72 0)
@@
 		(fields_autoplaced yes)
 		(effects
-			(font
-				(size 1.27 1.27)
-			)
-			(justify left bottom)
-		)
-	)
-	(label "SERVO"
-		(at 17.78 25.4 0)
-		(fields_autoplaced yes)
-		(effects
-			(font
-				(size 1.27 1.27)
-			)
-			(justify left bottom)
-		)
-	)
-	(label "OilTemp"
-		(at 17.78 34.29 0)
-		(fields_autoplaced yes)
-		(effects

Commit message: docs
Other:
- company: Jet & Aeronatucs Society -> Jet & Aeronautics Society
Changed lines of the file:
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@@
 		(date "2024-04-21")
 		(rev "0.1")
-		(company "Jet & Aeronatucs Society")
+		(company "Jet & Aeronautics Society")
 	)
 	(junction
