File: LOADCELL.kicad_sch (KiCad schematic)
At the start: 11 parts, among them J15 Conn_01x04_Socket, Q2 S8550M-D, U13 HX711

Commit message: docs
Other:
- company: (none) -> Jet & Aeronautics Society
Changed lines of the file:
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@@
 	(title_block
 		(date "2024-04-21")
+		(company "Jet & Aeronautics Society")
 	)
 	(junction
