File: max6675.kicad_sch (KiCad schematic)
At the start: 5 parts, among them CN8 DB910-7.62-2P, U8 MAX6675ISA+T

Commit message: docs
Other:
- company: (none) -> Jet & Aeronautics Society
Changed lines of the file:
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@@
 	(generator_version "8.0")
 	(paper "A4")
+	(title_block
+		(date "2024-04-21")
+		(company "Jet & Aeronautics Society")
+	)
 	(junction
 		(at 57.15 59.69)
